Commit message: - Implémentation de la création de multibody avec des links et de jointures dans UrdfEditor. - Créations de Shapes comme les spheres et les box.

File: test.urdf (robot description, URDF)
Before this commit: robot , 2 links, 1 joints
Links:
- removed link L1
- removed link L2
- added link B1, mass 1.00000; collision box size=1.00000 1.00000 1.00000; visual box size=1.00000 1.00000 1.00000
- added link B2, mass 1.00000; collision box size=1.00000 1.00000 1.00000; visual box size=1.00000 1.00000 1.00000
- added link S1, mass 1.00000; collision sphere radius=0.75000; visual sphere radius=0.75000
Joints:
- removed joint Joint
- added joint B1S1: type continuous, parent B1, child S1, origin xyz=0.00000 0.00000 0.50000 rpy=0.00000 0.00000 0.00000, axis 1.00000 0.00000 0.00000
- added joint S1B2: type continuous, parent S1, child B2, origin xyz=0.00000 0.00000 0.50000 rpy=0.00000 0.00000 0.00000, axis 0.00000 1.00000 0.00000

Commit message: Remplacement de createMultibody avec une génération de fichier URDF et son chargement pour supporter les jointures sphériques.

File: test.urdf (robot description, URDF)
Before this commit: robot , 3 links, 2 joints
Links:
- removed link S1
- link B1: mass 1.00000 -> 1
- link B2: mass 1.00000 -> 1
Joints:
- removed joint B1S1
- removed joint S1B2
- added joint J1: type spherical, parent B1, child B2, origin xyz=0.00000 0.00000 1.50000 rpy=0.00000 0.00000 0.00000, axis 1.00000 0.00000 0.00000

Commit message: Utilisation de deux jointures revolute pour relier un membre. Ajout d'un moteur.

File: test.urdf (robot description, URDF)
Before this commit: robot , 2 links, 1 joints
Links:
- added link S1, mass 1; collision sphere radius=0.5; visual sphere radius=0.5
Joints:
- removed joint J1
- added joint B1S1: type continuous, parent B1, child S1, origin xyz=0.00000 0.00000 0.50000 rpy=0.00000 0.00000 0.00000, axis 1.00000 0.00000 0.00000
- added joint S1B2: type continuous, parent S1, child B2, origin xyz=0.00000 0.00000 0.50000 rpy=0.00000 0.00000 0.00000, axis 0.00000 1.00000 0.00000

Commit message: Actuation simple de jointures.

File: test.urdf (robot description, URDF)
Before this commit: robot , 3 links, 2 joints
Joints:
- joint B1S1: limit (none) -> lower=-0.7854 upper=0.7854 effort=1000.0 velocity=0.5; type continuous -> revolute
- joint S1B2: limit (none) -> lower=-0.5236 upper=0.5236 effort=1000.0 velocity=0.5; type continuous -> revolute

Commit message: Déplacement du centre de rotation de la jointure vers une position plus correcte.

File: test.urdf (robot description, URDF)
Before this commit: robot , 3 links, 2 joints
Joints:
- joint S1B2: origin xyz=0.00000 0.00000 0.50000 rpy=0.00000 0.00000 0.00000 -> xyz=0.00000 0.00000 0.00000 rpy=0.00000 0.00000 0.00000
