Commit message: Refactorisation du code de création de fichiers Urdf en orienté objet.

File: data/Creature.urdf (robot description, URDF)
Before this commit: robot , 7 links, 6 joints
Links:
- link Base: mass 1 -> 1.00000
- link Limb1: mass 1 -> 1.00000
- link Limb2: mass 1 -> 1.00000
- link Limb3: mass 1 -> 1.00000
- link S_Base/Limb1: mass 1 -> 1.00000; geometry collision sphere radius=0.50000; visual sphere radius=0.50000
- link S_Base/Limb2: mass 1 -> 1.00000; geometry collision sphere radius=0.50000; visual sphere radius=0.50000
- link S_Base/Limb3: mass 1 -> 1.00000; geometry collision sphere radius=0.50000; visual sphere radius=0.50000

Commit message: - Les créatures peuvent maintenant être nommées. - Les créatures utilisent désormait des limites qui vont de pi à -pi par défaut.

File: data/Creature.urdf (robot description, URDF)
Before this commit: robot robot, 7 links, 6 joints
Joints:
- joint Jx_Base/Limb1: limit (none) -> lower=-3.14159 upper=3.14159 effort=1000.0 velocity=0.5; type continuous -> revolute
- joint Jx_Base/Limb2: limit (none) -> lower=-3.14159 upper=3.14159 effort=1000.0 velocity=0.5; type continuous -> revolute
- joint Jx_Base/Limb3: limit (none) -> lower=-3.14159 upper=3.14159 effort=1000.0 velocity=0.5; type continuous -> revolute
- joint Jy_Base/Limb1: limit (none) -> lower=-3.14159 upper=3.14159 effort=1000.0 velocity=0.5; type continuous -> revolute
- joint Jy_Base/Limb2: limit (none) -> lower=-3.14159 upper=3.14159 effort=1000.0 velocity=0.5; type continuous -> revolute
- joint Jy_Base/Limb3: limit (none) -> lower=-3.14159 upper=3.14159 effort=1000.0 velocity=0.5; type continuous -> revolute

Commit message: Création de la classe d'évolution et amélioration de la classe créature pour pouvoir spécifier sa racine.

File: data/Creature.urdf (robot description, URDF)
Before this commit: robot Creature, 7 links, 6 joints
Links:
- removed link Base
- removed link Limb1
- removed link Limb2
- removed link Limb3
- removed link S_Base/Limb1
- removed link S_Base/Limb2
- removed link S_Base/Limb3
- added link B1, mass 1.00000; collision box size=1.00000 1.00000 1.00000; visual box size=1.00000 1.00000 1.00000
- added link B2, mass 1.00000; collision box size=1.00000 1.00000 1.00000; visual box size=1.00000 1.00000 1.00000
- added link S_B1/B2, mass 1.00000; collision sphere radius=0.50000; visual sphere radius=0.50000
Joints:
- removed joint Jx_Base/Limb1
- removed joint Jx_Base/Limb2
- removed joint Jx_Base/Limb3
- removed joint Jy_Base/Limb1
- removed joint Jy_Base/Limb2
- removed joint Jy_Base/Limb3
- added joint Jx_B1/B2: type revolute, parent B1, child S_B1/B2, origin xyz=1.00000 0.00000 0.00000 rpy=0.00000 0.00000 0.00000, axis 1.00000 0.00000 0.00000, limit lower=-3.14159 upper=3.14159 effort=1000.0 velocity=0.5
- added joint Jy_B1/B2: type revolute, parent S_B1/B2, child B2, origin xyz=0.00000 0.00000 0.00000 rpy=0.00000 0.00000 0.00000, axis 0.00000 1.00000 0.00000, limit lower=-3.14159 upper=3.14159 effort=1000.0 velocity=0.5

Commit message: Motorisation des créature avec un mouvement en losange.

File: data/Creature.urdf (robot description, URDF)
Before this commit: robot Creature, 3 links, 2 joints
Links:
- added link B3, mass 1.00000; collision box size=1.00000 1.00000 1.00000; visual box size=1.00000 1.00000 1.00000
- added link S_B1/B3, mass 1.00000; collision sphere radius=0.50000; visual sphere radius=0.50000
Joints:
- removed joint Jx_B1/B2
- added joint Jy_B1/B3: type revolute, parent S_B1/B3, child B3, origin xyz=0.00000 0.00000 0.00000 rpy=0.00000 0.00000 0.00000, axis 0.00000 1.00000 0.00000, limit lower=-3.14159 upper=3.14159 effort=1000.0 velocity=0.5
- added joint Jz_B1/B2: type revolute, parent B1, child S_B1/B2, origin xyz=1.00000 0.00000 0.00000 rpy=0.00000 0.00000 0.00000, axis 0.00000 0.00000 1.00000, limit lower=-3.14159 upper=3.14159 effort=1000.0 velocity=0.5
- added joint Jz_B1/B3: type revolute, parent B1, child S_B1/B3, origin xyz=-1.00000 0.00000 0.00000 rpy=0.00000 0.00000 0.00000, axis 0.00000 0.00000 1.00000, limit lower=-3.14159 upper=3.14159 effort=1000.0 velocity=0.5
